File: tavelan-mini-rc2014.kicad_pcb (KiCad board)
At the start: 2 copper layers, 132 x 112 mm, 4 parts

Commit message: V1 to JLCPCB
Parts:
- added C1: 0.1µF, Capacitor_THT:C_Disc_D5.0mm_W2.5mm_P5.00mm, F.Cu at (99.1, 85.0)
- added C2: 0.1µF, Capacitor_THT:C_Disc_D5.0mm_W2.5mm_P5.00mm, F.Cu at (114.3, 85.0)
- added C3: 0.1µF, Capacitor_THT:C_Disc_D5.0mm_W2.5mm_P5.00mm, F.Cu at (129.5, 85.0)
- added C4: 0.1µF, Capacitor_THT:C_Disc_D5.0mm_W2.5mm_P5.00mm, F.Cu at (144.8, 85.1)
- added C5: 0.1µF, Capacitor_THT:C_Disc_D5.0mm_W2.5mm_P5.00mm, F.Cu at (160.0, 85.0)
- added C6: 0.1µF, Capacitor_THT:C_Disc_D5.0mm_W2.5mm_P5.00mm, F.Cu at (175.3, 85.0)
- added C7: 0.1µF, Capacitor_THT:C_Disc_D5.0mm_W2.5mm_P5.00mm, F.Cu at (190.5, 85.1)
- added C8: 0.1µF, Capacitor_THT:C_Disc_D5.0mm_W2.5mm_P5.00mm, F.Cu at (203.3, 130.2)
- added C99: 220µF, Capacitor_THT:CP_Radial_D8.0mm_P3.80mm, F.Cu at (203.9, 120.0)
- added D1: LED, LED_THT:LED_D3.0mm, F.Cu at (205.1, 65.4)
- added J1: Alternate_Reset, TerminalBlock_TE-Connectivity:TerminalBlock_TE_282834-2_1x02_P2.54mm_Horizontal, F.Cu at (203.8, 74.9)
- added J2: Regulated_Power, TerminalBlock_TE-Connectivity:TerminalBlock_TE_282834-2_1x02_P2.54mm_Horizontal, F.Cu at (203.8, 108.6)
- added R1: 4.7kΩ, Resistor_THT:R_Axial_DIN0207_L6.3mm_D2.5mm_P10.16mm_Horizontal, F.Cu at (204.5, 102.9)
- added R2: 560Ω, Resistor_THT:R_Axial_DIN0207_L6.3mm_D2.5mm_P10.16mm_Horizontal, F.Cu at (208.3, 102.9)
- added SW1: Reset, Button_Switch_THT:SW_PUSH_6mm, F.Cu at (203.8, 88.9)
- added U1: ~, Connector_PinSocket_2.54mm:PinSocket_1x40_P2.54mm_Vertical, F.Cu at (91.4, 40.6)
- added U2: ~, Connector_PinSocket_2.54mm:PinSocket_1x40_P2.54mm_Vertical, F.Cu at (106.7, 40.6)
- added U3: ~, Connector_PinSocket_2.54mm:PinSocket_1x40_P2.54mm_Vertical, F.Cu at (121.9, 40.6)
- added U4: ~, Connector_PinSocket_2.54mm:PinSocket_1x40_P2.54mm_Vertical, F.Cu at (137.2, 40.6)
- added U5: ~, Connector_PinSocket_2.54mm:PinSocket_1x40_P2.54mm_Vertical, F.Cu at (152.4, 40.6)
- added U6: ~, Connector_PinSocket_2.54mm:PinSocket_1x40_P2.54mm_Vertical, F.Cu at (167.6, 40.6)
- added U7: ~, Connector_PinSocket_2.54mm:PinSocket_1x40_P2.54mm_Vertical, F.Cu at (182.9, 40.6)
- added U8: ~, Connector_PinSocket_2.54mm:PinSocket_1x40_P2.54mm_Vertical, F.Cu at (198.1, 40.6)
Routing:
- net +5V: track 0.00 -> 223.0 mm
- net GND: track 0.00 -> 189.6 mm
- net /~{RESET}: track 0.00 -> 136.6 mm, vias 0 -> 1
- net /a0: track 0.00 -> 111.6 mm
- net /~{M1}: track 0.00 -> 111.6 mm
- net /~{WR}: track 0.00 -> 106.7 mm
- net /~{RD}: track 0.00 -> 106.7 mm
- net /~{MREQ}: track 0.00 -> 106.7 mm
- net /~{IORQ}: track 0.00 -> 106.7 mm
- net /~{INT}: track 0.00 -> 106.7 mm
- net /d7: track 0.00 -> 106.7 mm
- net /d6: track 0.00 -> 106.7 mm
- net /d5: track 0.00 -> 106.7 mm
- net /d4: track 0.00 -> 106.7 mm
- net /d3: track 0.00 -> 106.7 mm
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Other:
- board text added: "+5V"
- board text added: "+5v"
- board text added: "Ext. Reset"
- board text added: "GND"
- board text added: "Official spec (3-slot backplane schems): 15.24mm between sockets"
- board text added: "Regulated Power"
- board text added: "TAVELAN BACKPLANE DESIGNED FOR RC2014"
- board text added: "a0"
- board text added: "a1"
- board text added: "a10"
- board text added: "a11"
- board text added: "a12"
- board text added: "a13"
- board text added: "a14"
- board text added: "a15"
- board text added: "a2"
- board text added: "a3"
- board text added: "a4"
- board text added: "a5"
- board text added: "a6"
- board text added: "a7"
- board text added: "a8"
- board text added: "a9"
- board text added: "clk"
- board text added: "d0"
- board text added: "d1"
- board text added: "d2"
- board text added: "d3"
- board text added: "d4"
- board text added: "d5"
- board text added: "d6"
- board text added: "d7"
- board text added: "gnd"
- board text added: "leadedsolder.com 2024 v1.0"
- board text added: "rx"
- board text added: "tx"
- board text added: "user1"
- board text added: "user2"
- board text added: "user3"
- board text added: "user4"
- board text added: "~{int}"
- board text added: "~{iorq}"
- board text added: "~{m1}"
- board text added: "~{mreq}"
- board text added: "~{rd}"
- board text added: "~{reset}"
- board text added: "~{wr}"

Commit message: Round tracks, of course
Routing:
- net +5V: track 223.0 -> 219.1 mm
- net /~{M1}: track 111.6 -> 108.9 mm
- net /a0: track 111.6 -> 108.9 mm
- net GND: track 189.6 -> 188.0 mm
