File: tavelan-mini-rc2014.kicad_pcb (KiCad board)
At the start: 2 copper layers, 132 x 112 mm, 27 parts, among them J1 Alternate_Reset, J2 Regulated_Power, SW1 Reset

Commit message: OSHW logo
Parts:
- added REF**: OSHW-Logo2_9.8x8mm_Copper, Symbol:OSHW-Logo2_9.8x8mm_Copper, F.Cu at (84.8, 133.1)
